Commit message: 22--10-24-URDF-setting-complete

File: urdf/spmr02.urdf (robot description, URDF)
Before this commit: robot spmr02, 5 links, 4 joints
Joints:
- joint left_wheel_joint: origin xyz=0 -0.40407 0 rpy=1.5708 0 1.5708 -> xyz=0 -0.40407 -0.001 rpy=1.5708 0 1.5708
- joint right_wheel_joint: origin xyz=0 0.40407 0 rpy=1.5708 0 -1.5708 -> xyz=0 0.40407 -0.001 rpy=1.5708 0 -1.5708
